File: PCB/MyPCB.kicad_sch (KiCad schematic)
At the start: 10 parts, among them J1 OLED_DISPLAY, SW1 SW_Push, SW2 SW_Push, SW3 SW_Push, SW4 SW_Push, U1 XIAO-RP2040-DIP

Commit message: finish case
Parts:
- SW1: renamed from SW4; footprint MXCHERRY:MX-Hotswap-1U -> Button_Switch_Keyboard:SW_Cherry_MX_1.00u_PCB
- SW2: renamed from SW3; footprint MXCHERRY:MX-Hotswap-1U -> Button_Switch_Keyboard:SW_Cherry_MX_1.00u_PCB
- SW3: renamed from SW2; footprint MXCHERRY:MX-Hotswap-1U -> Button_Switch_Keyboard:SW_Cherry_MX_1.00u_PCB
- SW4: renamed from SW1; footprint MXCHERRY:MX-Hotswap-1U -> Button_Switch_Keyboard:SW_Cherry_MX_1.00u_PCB
Changed lines of the file:
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@@
 		(dnp no)
 		(fields_autoplaced yes)
-		(property "Reference" "SW2"
+		(property "Reference" "SW3"
 			(at 72.39 90.17 0)
 			(effects
@@
 			)
 		)
-		(property "Footprint" "MXCHERRY:MX-Hotswap-1U"
+		(property "Footprint" "Button_Switch_Keyboard:SW_Cherry_MX_1.00u_PCB"
 			(at 72.39 92.71 0)
 			(effects
@@
 			(project "MyPCB"
 				(path "/66e1480d-47e5-42ab-a4f5-0aab8b02bd4f"
-					(reference "SW2")
+					(reference "SW3")
 					(unit 1)
 				)
@@
 		(dnp no)
 		(fields_autoplaced yes)
-		(property "Reference" "SW3"
+		(property "Reference" "SW2"
 			(at 72.39 100.33 0)
 			(effects
@@
 			)
 		)
-		(property "Footprint" "MXCHERRY:MX-Hotswap-1U"
+		(property "Footprint" "Button_Switch_Keyboard:SW_Cherry_MX_1.00u_PCB"
 			(at 72.39 102.87 0)
 			(effects
@@
 			(project "MyPCB"
 				(path "/66e1480d-47e5-42ab-a4f5-0aab8b02bd4f"
-					(reference "SW3")
+					(reference "SW2")
 					(unit 1)
 				)
@@
 		(dnp no)
 		(fields_autoplaced yes)
-		(property "Reference" "SW4"
+		(property "Reference" "SW1"
 			(at 72.39 111.76 0)
 			(effects
@@
 			)
 		)
-		(property "Footprint" "MXCHERRY:MX-Hotswap-1U"
+		(property "Footprint" "Button_Switch_Keyboard:SW_Cherry_MX_1.00u_PCB"
 			(at 72.39 114.3 0)
 			(effects
@@
 			(project "MyPCB"
 				(path "/66e1480d-47e5-42ab-a4f5-0aab8b02bd4f"
-					(reference "SW4")
+					(reference "SW1")
 					(unit 1)
 				)
@@
 		(dnp no)
 		(fields_autoplaced yes)
-		(property "Reference" "SW1"
+		(property "Reference" "SW4"
 			(at 72.39 80.01 0)
 			(effects
@@
 			)
 		)
-		(property "Footprint" "MXCHERRY:MX-Hotswap-1U"
+		(property "Footprint" "Button_Switch_Keyboard:SW_Cherry_MX_1.00u_PCB"
 			(at 72.39 82.55 0)
 			(effects
@@
 			(project ""
 				(path "/66e1480d-47e5-42ab-a4f5-0aab8b02bd4f"
-					(reference "SW1")
-					(unit 1)
-				)
+					(reference "SW4")
+					(unit 1)
+				)
